File: generalRGBmod/Main-PCB/v1/n64rgbv1.sch (EAGLE design)
At the start: 76 parts, among them U1 5M570ZT100C5, U2 THS7374, U3 TLV70018-DDC

Commit message: N64RGBv1/v2 misc updates  (thanks to iFixRetro for giving feedback here!!!): - bugfix BOM and silkscreen (N64RGBv2) - silkscreen update to distinguish between MaxII and MaxV setup avoiding assembly mistakes - move power regulator to BOT copper side (N64RGBv1) - additional jumper J1 to select between 240LE and 570LE CPLD (for proper usage of the 5M240ZT)
Parts:
- removed C33: 1u, rcl:C-EUC0603
- added C1A, C22A: (no value), rcl:C-EUC0805
- added C2, C3: 10u, rcl:C-EUC0805
- added FB2: (no value), rcl:R-EU_R0603
- C31: value 10u -> 1u; device rcl:C-EUC1206K -> rcl:C-EUC0603
Connections:
- new net VCCINT: C11.1, C13.1, J1.2, U1.VCCINT@2, U1.VCCINT@3
- net GND: now also C1A.2, C2.2, C22A.2, C3.2; no longer C33.2
- net N$54: now also C1A.1
- net VCC@1.8V: now also C3.1, C32.1, FB2.2, J1.1; no longer C11.1, C13.1, C33.1, J1.2, U1.VCCINT@2, U1.VCCINT@3
- net VCC@3.3V: now also C2.1, C22A.1, FB2.1; no longer C32.1, J1.1
Other:
- moved on the sheet: C10, C11, C12, C13, C14, C15, C16, C17, C18, C19, C21, C31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
